Commit message: 2026.6.14 更新 1. 改造原仿真小车及仿真世界，引入mid360仿真激光雷达 2. 删除cartographer建图算法 3. 增加fastlio2全局重定位包 4. 接入fastlio2建图算法

File: src/description/urdf/robot.urdf (robot description, URDF)
Before this commit: robot car_robot, 2 links, 1 joints
Links:
- added link base_footprint
- added link camera_link, mass 0.01; collision box size=0.02 0.10 0.02; visual box size=0.02 0.10 0.02
- added link camera_optical_link
- added link front_left_wheel_link, mass 0.18; collision cylinder length=0.045 radius=0.055; visual cylinder length=0.045 radius=0.055
- added link front_right_wheel_link, mass 0.18; collision cylinder length=0.045 radius=0.055; visual cylinder length=0.045 radius=0.055
- added link mid360, mass 0.1; visual box size=0.1 0.06 0.06
- added link rear_left_wheel_link, mass 0.18; collision cylinder length=0.045 radius=0.055; visual cylinder length=0.045 radius=0.055
- added link rear_right_wheel_link, mass 0.18; collision cylinder length=0.045 radius=0.055; visual cylinder length=0.045 radius=0.055
- link base_link: mass None -> 1.8; geometry collision box size=0.42 0.28 0.1; visual box size=0.42 0.28 0.1
- link imu_link: mass None -> 0.01; geometry collision box size=0.02 0.02 0.02; visual box size=0.02 0.02 0.02
Joints:
- added joint base_footprint_joint: type fixed, parent base_footprint, child base_link, origin xyz=0.0 0.0 0.10200000000000001 rpy=0.0 0.0 0.0
- added joint camera_joint: type fixed, parent base_link, child camera_link, origin xyz=0.20 0.0 0.060 rpy=0.0 0.0 0.0
- added joint camera_optical_joint: type fixed, parent camera_link, child camera_optical_link, origin xyz=0 0 0 rpy=-1.5707963267948966 0.0 -1.5707963267948966
- added joint front_left_wheel_joint: type continuous, parent base_link, child front_left_wheel_link, origin xyz=0.145 0.165 -0.047 rpy=0.0 0.0 0.0, axis 0.0 1.0 0.0
- added joint front_right_wheel_joint: type continuous, parent base_link, child front_right_wheel_link, origin xyz=0.145 -0.165 -0.047 rpy=0.0 0.0 0.0, axis 0.0 1.0 0.0
- added joint mid360_joint: type fixed, parent base_link, child mid360, origin xyz=0.0 0.0 0.080 rpy=0.0 0.0 0.0
- added joint rear_left_wheel_joint: type continuous, parent base_link, child rear_left_wheel_link, origin xyz=-0.145 0.165 -0.047 rpy=0.0 0.0 0.0, axis 0.0 1.0 0.0
- added joint rear_right_wheel_joint: type continuous, parent base_link, child rear_right_wheel_link, origin xyz=-0.145 -0.165 -0.047 rpy=0.0 0.0 0.0, axis 0.0 1.0 0.0
- joint imu_joint: origin xyz=0.0 0.0 0.03 rpy=0.0 0.0 0.0 -> xyz=0.0 0.0 0.065 rpy=0.0 0.0 0.0

File: src/description/xacro/base.urdf.xacro (robot description, xacro)
@@ -2,6 +2,5 @@
 <robot xmlns:xacro="http://www.ros.org/wiki/xacro">
     <xacro:include filename="$(find description)/xacro/common_inertia.xacro"/>
-    <xacro:macro name="base_xacro" params="length radius">
-        <link name="base_footprint"/>
+    <xacro:macro name="base_xacro" params="length width height wheel_radius">
         <link name="base_link">
             <!-- 部件的外观描述-->
@@ -11,5 +10,5 @@
                 <!-- 几何形状-->
                 <geometry>
-                    <cylinder radius="${radius}" length="${length}"/>
+                    <box size="${length} ${width} ${height}"/>
                 </geometry>
                 <!-- 材质颜色-->
@@ -23,5 +22,5 @@
                 <!-- 几何形状-->
                 <geometry>
-                    <cylinder radius="${radius}" length="${length}"/>
+                    <box size="${length} ${width} ${height}"/>
                 </geometry>
                 <!-- 材质颜色-->
@@ -30,11 +29,6 @@
                 </material>
             </collision>
-            <xacro:cylinder_inertia m="1.0" r="${radius}" h="${length}"/>
+            <xacro:box_inertia m="1.8" w="${length}" h="${width}" d="${height}"/>
         </link>
-        <joint name="joint_name" type="fixed">
-            <origin xyz="0.0 0.0 ${length/2.0+0.032-0.001}" rpy="0.0 0.0 0.0"/>
-            <parent link="base_footprint"/>
-            <child link="base_link"/>
-        </joint>
     </xacro:macro>
 </robot>

File: src/description/xacro/gazebo_sensor_plugin.xacro (robot description, xacro)
@@ -1,86 +1,4 @@
 <?xml version="1.0"?>
 <robot xmlns:xacro="http://www.ros.org/wiki/xacro">
-    <xacro:macro name="gazebo_sensor_plugin">
-        <!-- <gazebo reference="laser_link">
-            <sensor name="laserscan" type="ray">
-                <plugin name="laserscan" filename="libgazebo_ros_ray_sensor.so">
-                    <ros>
-                        <namespace>/</namespace>
-                        <remapping>~/out:=scan</remapping>
-                    </ros>
-                    <output_type>sensor_msgs/LaserScan</output_type>
-                    <frame_name>laser_link</frame_name>
-                </plugin>
-                <always_on>true</always_on>
-                <visualize>true</visualize>
-                <update_rate>100</update_rate>
-                <pose>0 0 0 0 0 0</pose>
-                <ray>
-                    <scan>
-                        <horizontal>
-                            <samples>360</samples>
-                            <resolution>1.000000</resolution>
-                            <min_angle>0.000000</min_angle>
-                            <max_angle>6.280000</max_angle>
-                        </horizontal>
-                    </scan>
-                    <range>
-                        <min>0.120000</min>
-                        <max>8.0</max>
-                        <resolution>0.015000</resolution>
-                    </range>
-                    <noise>
-                        <type>gaussian</type>
-                        <mean>0.0</mean>
-                        <stddev>0.01</stddev>
-                    </noise>
-                </ray>
-            </sensor>
-        </gazebo> -->
-        <gazebo reference="laser_link">
-            <sensor name="velodyne-VLP16" type="ray">
-            <pose>0 0 0 0 0 0</pose>
-            <visualize>false</visualize>
-            <update_rate>10</update_rate>
-            <ray>
-                <scan>
-                <horizontal>
-                    <samples>440</samples>
-                    <resolution>1</resolution>
-                    <min_angle>-3.141592653589793</min_angle>
-                    <max_angle>3.141592653589793</max_angle>
-                </horizontal>
-                <vertical>
-                    <samples>16</samples>
-                    <resolution>1</resolution>
-                    <min_angle>-0.2617993877991494</min_angle>
-                    <max_angle> 0.2617993877991494</max_angle>
-                </vertical>
-                </scan>
-                <range>
-                <min>0.3</min>
-                <max>131.0</max>
-                <resolution>0.001</resolution>
-                </range>
-                <noise>
-                <type>gaussian</type>
-                <mean>0.0</mean>
-                <stddev>0.0</stddev>
-                </noise>
-            </ray>
-            <plugin filename="libgazebo_ros_velodyne_laser.so" name="gazebo_ros_laser_controller">
-                <ros>
-                <namespace>/</namespace>
-                <remapping>~/out:=velodyne_points</remapping>
-                </ros>
-                <frame_name>laser_link</frame_name>
-                <organize_cloud>false</organize_cloud>
-                <min_range>0.9</min_range>
-                <max_range>130.0</max_range>
-                <gaussian_noise>0.008</gaussian_noise>
-            </plugin>
-            </sensor>
-        </gazebo>
-    </xacro:macro>
     <gazebo reference="imu_link">
         <sensor name="imu_sensor" type="imu">
@@ -90,4 +8,5 @@
                 <remapping>~/out:=imu</remapping>
             </ros>
+            <frame_name>imu_link</frame_name>
             <initial_orientation_as_reference>false</initial_orientation_as_reference>
         </plugin>
@@ -153,16 +72,24 @@
 <gazebo reference="camera_link">
     <sensor type="depth" name="camera_sensor">
+        <visualize>false</visualize>
         <plugin name="depth_camera" filename="libgazebo_ros_camera.so">
             <frame_name>camera_optical_link</frame_name>
+            <camera_name>camera_sensor</camera_name>
+            <min_depth>0.15</min_depth>
+            <max_depth>15.0</max_depth>
         </plugin>
-        <always_on>true</always_on>
-        <update_rate>10</update_rate>
+        <always_on>false</always_on>
+        <update_rate>5</update_rate>
         <camera name="camera">
             <horizontal_fov>1.5009831567</horizontal_fov>
             <image>
-                <width>800</width>
-                <height>600</height>
+                <width>320</width>
+                <height>240</height>
                 <format>R8G8B8</format>
             </image>
+            <clip>
+                <near>0.15</near>
+                <far>15.0</far>
+            </clip>
             <distortion>
                 <k1>0.0</k1>

File: src/description/xacro/robot.urdf.xacro (robot description, xacro)
@@ -4,18 +4,26 @@
     <xacro:include filename="$(find description)/xacro/imu.urdf.xacro"/>
     <xacro:include filename="$(find description)/xacro/camera.urdf.xacro"/>
-    <xacro:include filename="$(find description)/xacro/laser.urdf.xacro"/>
     <xacro:include filename="$(find description)/xacro/wheel.urdf.xacro"/>
-    <xacro:include filename="$(find description)/xacro/caster.urdf.xacro"/>
     <xacro:include filename="$(find description)/xacro/gazebo_sensor_plugin.xacro"/>
     <xacro:include filename="$(find description)/xacro/ros2_control.xacro"/>
-    <xacro:base_xacro length="0.12" radius="0.10"/>
-    <xacro:imu_xacro xyz="0.0 0.0 0.02"/>
-    <xacro:camera_xacro xyz="0.10 0.0 0.075"/>
-    <xacro:laser_xacro xyz="0.0 0.0 0.10"/>
-    <xacro:wheel_xacro wheel_name="left_wheel" xyz="0.0 0.10 -0.06"/>
-    <xacro:wheel_xacro wheel_name="right_wheel" xyz="0.0 -0.10 -0.06"/>
-    <xacro:caster_xacro caster_name="front_caster" xyz="0.08 0.0 -0.076"/>
-    <xacro:caster_xacro caster_name="back_caster" xyz="-0.08 0.0 -0.076"/>
-    <xacro:gazebo_sensor_plugin />
+    <xacro:include filename="$(find ros2_livox_simulation)/urdf/mid360.xacro"/>
+    <xacro:property name="base_length" value="0.42"/>
+    <xacro:property name="base_width" value="0.28"/>
+    <xacro:property name="base_height" value="0.10"/>
+    <xacro:property name="wheel_radius" value="0.055"/>
+    <xacro:property name="wheel_width" value="0.045"/>
+    <xacro:property name="wheel_x" value="0.145"/>
+    <xacro:property name="wheel_y" value="0.165"/>
+    <xacro:property name="wheel_z" value="-0.047"/>
+    <xacro:base_xacro length="${base_length}" width="${base_width}" height="${base_height}" wheel_radius="${wheel_radius}"/>
+    <xacro:imu_xacro xyz="0.0 0.0 0.065"/>
+    <xacro:camera_xacro xyz="0.20 0.0 0.060"/>
+    <xacro:mid360 name="livox_frame" parent="base_link" topic="/livox/lidar">
+        <origin xyz="0.0 0.0 0.080" rpy="0.0 0.0 0.0"/>
+    </xacro:mid360>
+    <xacro:wheel_xacro wheel_name="front_left_wheel" xyz="${wheel_x} ${wheel_y} ${wheel_z}" radius="${wheel_radius}" width="${wheel_width}"/>
+    <xacro:wheel_xacro wheel_name="front_right_wheel" xyz="${wheel_x} ${-wheel_y} ${wheel_z}" radius="${wheel_radius}" width="${wheel_width}"/>
+    <xacro:wheel_xacro wheel_name="rear_left_wheel" xyz="${-wheel_x} ${wheel_y} ${wheel_z}" radius="${wheel_radius}" width="${wheel_width}"/>
+    <xacro:wheel_xacro wheel_name="rear_right_wheel" xyz="${-wheel_x} ${-wheel_y} ${wheel_z}" radius="${wheel_radius}" width="${wheel_width}"/>
     <xacro:ros2_control />
 </robot>

File: src/description/xacro/ros2_control.xacro (robot description, xacro)
@@ -6,12 +6,12 @@
                 <plugin>gazebo_ros2_control/GazeboSystem</plugin>
             </hardware>
-            <joint name="left_wheel_joint">
+            <joint name="front_left_wheel_joint">
                 <command_interface name="velocity">
-                    <param name="min">-1</param>
-                    <param name="max">1</param>
+                    <param name="min">-12</param>
+                    <param name="max">12</param>
                 </command_interface>
                 <command_interface name="effort">
-                    <param name="min">-0.1</param>
-                    <param name="max">0.1</param>
+                    <param name="min">-8.0</param>
+                    <param name="max">8.0</param>
                 </command_interface>
                 <state_interface name="position" />
@@ -19,12 +19,38 @@
                 <state_interface name="effort" />
             </joint>
-            <joint name="right_wheel_joint">
+            <joint name="front_right_wheel_joint">
                 <command_interface name="velocity">
-                    <param name="min">-1</param>
-                    <param name="max">1</param>
+                    <param name="min">-12</param>
+                    <param name="max">12</param>
                 </command_interface>
                 <command_interface name="effort">
-                    <param name="min">-0.1</param>
-                    <param name="max">0.1</param>
+                    <param name="min">-8.0</param>
+                    <param name="max">8.0</param>
+                </command_interface>
+                <state_interface name="position" />
+                <state_interface name="velocity" />
+                <state_interface name="effort" />
+            </joint>
+            <joint name="rear_left_wheel_joint">
+                <command_interface name="velocity">
+                    <param name="min">-12</param>
+                    <param name="max">12</param>
+                </command_interface>
+                <command_interface name="effort">
+                    <param name="min">-8.0</param>
+                    <param name="max">8.0</param>
+                </command_interface>
+                <state_interface name="position" />
+                <state_interface name="velocity" />
+                <state_interface name="effort" />
+            </joint>
+            <joint name="rear_right_wheel_joint">
+                <command_interface name="velocity">
+                    <param name="min">-12</param>
+                    <param name="max">12</param>
+                </command_interface>
+                <command_interface name="effort">
+                    <param name="min">-8.0</param>
+                    <param name="max">8.0</param>
                 </command_interface>
                 <state_interface name="position" />
@@ -41,5 +67,5 @@
             </ros>
         </plugin>
-</gazebo>
+    </gazebo>
     </xacro:macro>
 </robot>

File: src/description/xacro/wheel.urdf.xacro (robot description, xacro)
@@ -2,5 +2,5 @@
 <robot xmlns:xacro="http://www.ros.org/wiki/xacro">
     <xacro:include filename="$(find description)/xacro/common_inertia.xacro"/>
-    <xacro:macro name="wheel_xacro" params="wheel_name xyz">
+    <xacro:macro name="wheel_xacro" params="wheel_name xyz radius:=0.055 width:=0.045 mass:=0.18">
         <link name="${wheel_name}_link">
             <!-- 部件的外观描述-->
@@ -10,5 +10,5 @@
                 <!-- 几何形状-->
                 <geometry>
-                    <cylinder radius="0.032" length="0.04"/>
+                    <cylinder radius="${radius}" length="${width}"/>
                 </geometry>
                 <!-- 材质颜色-->
@@ -22,5 +22,5 @@
                 <!-- 几何形状-->
                 <geometry>
-                    <cylinder radius="0.032" length="0.04"/>
+                    <cylinder radius="${radius}" length="${width}"/>
                 </geometry>
                 <!-- 材质颜色-->
@@ -29,5 +29,5 @@
                 </material>
             </collision>
-            <xacro:cylinder_inertia m="0.1" r="0.032" h="0.04"/>
+            <xacro:cylinder_inertia m="${mass}" r="${radius}" h="${width}"/>
         </link>
         <joint name="${wheel_name}_joint" type="continuous">
@@ -38,8 +38,11 @@
         </joint>
         <gazebo reference="${wheel_name}_link">
-            <mu1 value="20.0"/>
-            <mu2 value="20.0"/>
-            <kp value="1000000000.0"/>
-            <kd value="1.0"/>
+            <fdir1>1 0 0</fdir1>
+            <mu1>8.0</mu1>
+            <mu2>0.35</mu2>
+            <kp>100000.0</kp>
+            <kd>1.0</kd>
+            <maxVel>0.1</maxVel>
+            <minDepth>0.001</minDepth>
         </gazebo>
     </xacro:macro>

File: src/livox_laser_simulation_RO2/urdf/mid360.xacro (robot description, xacro)
@@ -4,5 +4,5 @@
   <xacro:property name="laser_min_range" value="0.1"/>
   <xacro:property name="laser_max_range" value="200.0"/>
-  <xacro:property name="samples" value="40000"/>
+  <xacro:property name="samples" value="12000"/>
   <xacro:property name="resolution" value="0.002"/>
   <xacro:property name="noise_mean" value="0.0"/>
