Commit message: 2026.6.14 第二次更新 1. 加入了地形分析包并接入了项目 2. 增加了分析地形分析包输出点云话题的脚本 3. 接入了nav2导航 4. 增加了3d转2d的地图工具包 5. 增加了地形分析包用的数据对齐接口包 6. 增加了nav2导航新恢复行为，代替后退 7. 修改了行为树

File: src/livox_laser_simulation_RO2/urdf/mid360.xacro (robot description, xacro)
@@ -4,5 +4,5 @@
   <xacro:property name="laser_min_range" value="0.1"/>
   <xacro:property name="laser_max_range" value="200.0"/>
-  <xacro:property name="samples" value="12000"/>
+  <xacro:property name="samples" value="10000"/>
   <xacro:property name="resolution" value="0.002"/>
   <xacro:property name="noise_mean" value="0.0"/>

Commit message: 2026.6.21 更新 1. 在仿真world世界里加入了楼梯 2. 加入了自己写的地形分析包 3. 调整了lio_interface中被转换的点云话题 4. 修改了仿真雷达的采样点数

File: src/livox_laser_simulation_RO2/urdf/mid360.xacro (robot description, xacro)
@@ -4,5 +4,5 @@
   <xacro:property name="laser_min_range" value="0.1"/>
   <xacro:property name="laser_max_range" value="200.0"/>
-  <xacro:property name="samples" value="10000"/>
+  <xacro:property name="samples" value="30000"/>
   <xacro:property name="resolution" value="0.002"/>
   <xacro:property name="noise_mean" value="0.0"/>
