Commit message: 2026.7.6 更新 1. 恢复mid360采样率 2. 全局规划器和控制器恢复默认

File: src/livox_laser_simulation_RO2/urdf/mid360.xacro (robot description, xacro)
@@ -4,5 +4,5 @@
   <xacro:property name="laser_min_range" value="0.1"/>
   <xacro:property name="laser_max_range" value="200.0"/>
-  <xacro:property name="samples" value="30000"/>
+  <xacro:property name="samples" value="40000"/>
   <xacro:property name="resolution" value="0.002"/>
   <xacro:property name="noise_mean" value="0.0"/>
